Commit message: remove hector control, adjust pai model

File: Hector_ROS_Simulation/pai_description/xacro/pai.urdf (robot description, URDF)
Before this commit: robot PAI-urdf, 11 links, 10 joints
Joints:
- joint L_calf_joint: limit (none) -> lower=-3 upper=3 effort=33.5 velocity=21; type continuous -> revolute
- joint L_hip2_joint: limit (none) -> lower=-3 upper=3 effort=33.5 velocity=21; type continuous -> revolute
- joint L_hip_joint: limit (none) -> lower=-3 upper=3 effort=33.5 velocity=21; type continuous -> revolute
- joint L_thigh_joint: limit (none) -> lower=-3 upper=3 effort=33.5 velocity=21; type continuous -> revolute
- joint L_toe_joint: limit (none) -> lower=-3 upper=3 effort=33.5 velocity=21; type continuous -> revolute
- joint R_calf_joint: limit (none) -> lower=-3 upper=3 effort=33.5 velocity=21; type continuous -> revolute
- joint R_hip2_joint: limit (none) -> lower=-3 upper=3 effort=33.5 velocity=21; type continuous -> revolute
- joint R_hip_joint: limit (none) -> lower=-3 upper=3 effort=33.5 velocity=21; type continuous -> revolute
- joint R_thigh_joint: limit (none) -> lower=-3 upper=3 effort=33.5 velocity=21; type continuous -> revolute
- joint R_toe_joint: limit (none) -> lower=-3 upper=3 effort=33.5 velocity=21; type continuous -> revolute
